File: PCB/KiCAD/goob/goob.kicad_pcb (KiCad board)
At the start: 2 copper layers, 125.5 x 90.3 mm, 109 parts, among them J1 Conn_01x06_Female, J11 Conn_01x02, J14 Conn_01x06, J15 Conn_01x06, J2 Conn_01x02, J3 Conn_01x02, J4 Conn_01x01, J5 Rumble, J6 Conn_01x06, J8 USB_B_Micro, Q1 Q_NMOS_GSD, Q2 Q_PMOS_GDS, Q3 Q_NMOS_GSD, SW1 A, SW10 Dup, SW11 Dright, SW12 Ddown, SW2 B, SW3 X, SW4 Y, SW5 Start, SW6 L, SW7 R, SW8 Z, SW9 Dleft, U1 MCP3202, U12 USBLC6-2P6, U13 USBLC6-2P6, U2 2x DRV5053CAQLPGM Hall Effect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, U3 MCP3202, U4 DRV5055A3xDBZxQ1, U5 Stickbox_Assembly_CStick, U6 AMS1117-3.3, U7 W25Q128JVS, U8 RP2040, U9 DRV5055A3xDBZxQ1, Y1 Crystal_GND24

Commit message: WIP
Parts:
- removed U4, U9: DRV5055A3xDBZxQ1, PhobGCC_2_0_0_footprints:SOT-23
- removed U5: Stickbox_Assembly_CStick, PhobGCC_2_0_0_footprints:GCC_Stickbox_Hall_Only
- added G*** (x2): LOGO, LOGO, F.Cu at (69.7, 51.1)
- added G***: LOGO, LOGO, B.Cu at (156.2, 69.1)
- moved U2 0.10 mm to (69.7, 51.1), turned to -2.899 degrees
- turned U2 to 90 degrees
Connections:
- U2 pad 13: (no net) -> /GND_C
- U2 pad 14: (no net) -> /H2XS
- U2 pad 15: (no net) -> VCC
- U2 pad 16: (no net) -> /GND_C
- U2 pad 17: (no net) -> /H2YS
- U2 pad 18: (no net) -> VCC
Routing:
- net /GND_C: track 15.8 -> 8.15 mm, vias 6 -> 4
- net /H2XS: track 23.2 -> 17.4 mm, vias 1 -> 0
- net VCC: track 11.6 -> 6.89 mm, vias 4 -> 2
- net /H2YS: track 16.9 -> 15.4 mm, vias 1 -> 0
Other:
- board text added: "goob DX"
- board text removed: "goob"

Commit message: New PC
Parts:
- removed H14: MouseBite, PhobGCC_2_0_0_footprints:breakaway-mousebites-double-v2-small
- removed J14, J15: Conn_01x06, PhobGCC_2_0_0_footprints:PinSocket_1x06_P2.00mm_Vertical
- added H15: MouseBite, PhobGCC_2_0_0_footprints:breakaway-mousebites-double-v2-large, F.Cu at (115.0, 62.6)
- added J1: Conn_01x04_Male, Connector_PinHeader_2.00mm:PinHeader_1x04_P2.00mm_Vertical, F.Cu at (167.9, 78.7)
- added J1: Conn_01x04_Male, Connector_PinHeader_2.00mm:PinHeader_1x04_P2.00mm_Vertical, F.Cu at (115.3, 68.8)
- moved U3 52.3 mm to (161.3, 70.1), turned to 135 degrees
- moved C32 48.4 mm to (155.7, 67.3), turned to 135 degrees
- moved G*** 13.1 mm to (160.3, 56.6)
- moved C5 7.70 mm to (121.6, 99.3)
- moved H11 7.70 mm to (113.7, 76.1)
- moved R3 7.70 mm to (115.5, 88.8)
- moved R4 7.70 mm to (125.6, 99.3)
- moved C4 7.70 mm to (115.5, 92.8)
- moved H10 7.70 mm to (109.2, 91.7)
- moved H12 7.70 mm to (123.7, 95.4)
- moved H13 7.70 mm to (123.7, 86.4)
- moved U2 7.70 mm to (123.7, 90.9)
Connections:
- C32 pad 1: VCC -> +3V3
- C32 pad 2: /GND_C -> GND
- U3 pad 1: /CS2_2 -> /CS2
- U3 pad 2: /C_x_filt -> CX
- U3 pad 3: /C_y_filt -> CY
- U3 pad 4: /GND_C -> GND
- U3 pad 5: /Din2 -> /Din
- U3 pad 6: /Dout2 -> /Dout
- U3 pad 7: /CLK2 -> /CLK
- U3 pad 8: VCC -> +3V3
Routing:
- net /CS2_2: track 22.1 -> 0.00 mm, vias 1 -> 0
- net /CLK: track 128.3 -> 113.8 mm, vias 2 -> 3
- net /CLK2: track 11.7 -> 0.00 mm
- net /CS2: track 94.4 -> 84.2 mm, vias 3 -> 2
- net /Dout2: track 8.94 -> 0.00 mm
- net GND: track 132.0 -> 140.8 mm, vias 49 -> 53
- net /Dout: track 127.9 -> 119.6 mm, vias 4 -> 5
- net CY: track 0.00 -> 7.87 mm
- net VCC: track 6.89 -> 0.00 mm, vias 2 -> 0
- net /Din2: track 6.81 -> 0.00 mm
- net CX: track 0.00 -> 6.70 mm
- net /C_y_filt: track 26.1 -> 29.8 mm
- net /Din: track 125.5 -> 122.0 mm, vias 4 -> 5
- net +3V3: track 63.9 -> 67.2 mm
- net +5V: track 159.0 -> 156.2 mm
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Other:
- board size 125.5 x 90.3 mm -> 125.5 x 82.6 mm
- board text removed: "github.com/PhobGCC"

Commit message: Zl
Zl
Parts:
- added ?: , , F.Cu at (58.9, 36.7)
- added ?: , , F.Cu at (55.3, 36.4)
- added SW8L: ZL, PhobGCC_2_0_0_footprints:Z_Switch_Edge_Omron, F.Cu at (60.8, 35.5)
Connections:
- J6 pad 2: /GPIO12 -> GND
- U8 pad 15: /GPIO12 -> /LeftZ
Routing:
- net /LeftZ: track 0.00 -> 59.3 mm, vias 0 -> 2
- net /GPIO12: track 16.8 -> 0.00 mm
- net GND: track 140.8 -> 139.4 mm
Other:
- outline, holes or cut-outs redrawn
